Commit message: Update p3at.urdf.xacro

File: p3at_gazebo/urdf/p3at.urdf.xacro (robot description, xacro)
@@ -54,5 +54,5 @@
       </inertial>
       <visual>
-        <origin xyz="0 0 0" rpy="0 1.57079632679 0"/>
+        <origin xyz="0 0 0" rpy="1.57079632679 0 0"/>
         <geometry>
           <cylinder radius="${wheel_radius}" length="${wheel_width}"/>
@@ -63,5 +63,5 @@
       </visual>
       <collision>
-        <origin xyz="0 0 0" rpy="0 1.57079632679 0"/>
+        <origin xyz="0 0 0" rpy="1.57079632679 0 0"/>
         <geometry>
           <cylinder radius="${wheel_radius}" length="${wheel_width}"/>
@@ -116,8 +116,7 @@
     <parent link="camera_link"/>
     <child link="camera_depth_optical_frame"/>
-    <!-- REP 103 optical frame: Z forward, X right, Y down -->
     <origin xyz="0 0 0" rpy="-1.57079632679 0 -1.57079632679"/>
   </joint>
-  <!-- Gazebo: friction and plugins -->
+  <!-- Gazebo: friction -->
   <gazebo reference="front_left_wheel_link">
     <mu1>1.0</mu1>
@@ -136,5 +135,5 @@
     <mu2>1.0</mu2>
   </gazebo>
-  <!-- Skid-steer drive plugin (preferred). If your system lacks this plugin, switch to libgazebo_ros_diff_drive.so. -->
+  <!-- Skid-steer drive plugin -->
   <gazebo>
     <plugin name="skid_steer_drive" filename="libgazebo_ros_skid_steer_drive.so">
@@ -155,8 +154,14 @@
     </plugin>
   </gazebo>
-  <!-- Depth camera plugin. Publishes:
-       /camera/depth (sensor_msgs/Image)
-       /camera/depth/camera_info (sensor_msgs/CameraInfo)
-       /camera/depth/points (sensor_msgs/PointCloud2) -->
+  <!-- Joint state publisher plugin (Gazebo -> /joint_states) -->
+  <gazebo>
+    <plugin name="joint_state_publisher" filename="libgazebo_ros_joint_state_publisher.so">
+      <robotNamespace>/</robotNamespace>
+      <jointName>front_left_wheel_joint, rear_left_wheel_joint, front_right_wheel_joint, rear_right_wheel_joint</jointName>
+      <updateRate>50</updateRate>
+      <alwaysOn>true</alwaysOn>
+    </plugin>
+  </gazebo>
+  <!-- Depth camera plugin -->
   <gazebo reference="camera_link">
     <sensor type="depth" name="depth_camera">
